Commit message: fix gravity problem, and PID issue

File: aww_description/urdf/anymal_with_wheels.urdf.xacro (robot description, xacro)
@@ -1,3 +1,9 @@
-<?xml version="1.0" ?>
+<?xml version="1.0" encoding="utf-8"?>
+<!-- =================================================================================== -->
+<!--   Copyright 2020 ANYbotics, https://www.anybotics.com                               -->
+<!-- =================================================================================== -->
+<!-- This version is an unofficial adapted version of the description of the ANYmal C    -->
+<!-- developed by ANYbotics. The repository with original files can be found in          -->
+<!-- https://github.com/ANYbotics/anymal_c_simple_description.                           -->
 <robot xmlns:sensor="http://playerstage.sourceforge.net/gazebo/xmlschema/#sensor"
        xmlns:controller="http://playerstage.sourceforge.net/gazebo/xmlschema/#controller"
@@ -5,10 +11,1719 @@
        xmlns:xacro="http://playerstage.sourceforge.net/gazebo/xmlschema/#xacro"
        name="aww" >
-  <xacro:include filename="$(find aww_description)/urdf/aww_macro.xacro"/>
-    <!-- Used for fixing robot to Gazebo -->
-    <link name="world"/>
-    <!-- robor -->
-    <xacro:aww_robot parent="world">
-        <origin xyz="0 0 0.4" rpy="0 0 0" /> <!--slightly above gazebo plane-->.
-    </xacro:aww_robot>
+<!-- =============================================================================== -->
+<!--  Xacro Properties                                                               -->
+<!-- =============================================================================== -->
+    <xacro:property name="PI" value="3.1415926535897931" />
+    <xacro:property name="wheel_radius" value="0.098" />
+    <xacro:property name="wheel_width" value="0.040" />
+<!-- =============================================================================== -->
+<!--  Define some macros                                                             -->
+<!-- =============================================================================== -->
+    <!-- MACRO TRANSMISSION USED IN THE JOINTS -->
+    <xacro:macro name="transmission_block" params="joint_name">
+        <transmission name="transmission">
+            <type>transmission_interface/SimpleTransmission</type>
+            <joint name="${joint_name}">
+                <!-- hardwareInterface>hardware_interface/PositionJointInterface</hardwareInterface -->
+                <!--hardwareInterface>hardware_interface/VelocityJointInterface</hardwareInterface-->
+                <hardwareInterface>hardware_interface/EffortJointInterface</hardwareInterface>
+            </joint>
+            <actuator name="${joint_name}_motor">
+                <hardwareInterface>hardware_interface/EffortJointInterface</hardwareInterface>
+                <mechanicalReduction>1</mechanicalReduction>
+            </actuator>
+        </transmission>
+    </xacro:macro>
+    <!-- MACRO USED TO CREATE WHEELS -->
+    <xacro:macro name="wheel" params="prefix *joint_pose">
+        <!-- first create a link for the wheel -->
+        <link name="${prefix}_wheel_link">
+            <visual>
+                <origin xyz="0 0 0" rpy="${pi/2} 0 0"/>
+                <geometry>
+                   <mesh filename="package://aww_description/meshes/jackal-wheel.stl" scale="0.9 0.9 0.9"/>
+                </geometry>
+                <material name="black" />
+            </visual>
+            <collision>
+                <origin xyz="0 0 0" rpy="${pi/2} 0 0"/>
+                <geometry>
+                    <cylinder radius="${wheel_radius}" length="${wheel_width}"/>
+                </geometry>
+            </collision>
+            <inertial>
+                <origin xyz="0 0 0" rpy="0 0 0"/>
+                <mass value="0.477"/>
+                <inertia
+                    ixx="0.0013" ixy="0" ixz="0"
+                    iyy="0.0024" iyz="0"
+                    izz="0.0013"/>
+            </inertial>
+        </link>
+        <!-- Create a gazebo configuration params -->
+        <gazebo reference="${prefix}_wheel_link">
+            <material>Gazebo/FlatBlack</material>
+            <selfCollide>false</selfCollide>
+            <mu1 value="0.5"/>
+            <mu2 value="0.5"/>
+            <kp value="10000000.0" />
+            <kd value="1" />
+            <fdir1 value="1 0 0"/>
+        </gazebo>
+        <!-- Create a joint for the links -->
+        <joint name="${prefix}_wheel" type="continuous">
+            <parent link="${prefix}_LEG"/>
+            <child link="${prefix}_wheel_link" />
+            <xacro:insert_block name="joint_pose" />
+            <axis xyz="0 1 0" />
+        </joint>
+        <!-- Link the join to a transmission (used in control) -->
+        <transmission name="${prefix}_wheel_trans">
+            <type>transmission_interface/SimpleTransmission</type>
+            <joint name="${prefix}_wheel">
+                <hardwareInterface>hardware_interface/VelocityJointInterface</hardwareInterface>
+            </joint>
+            <actuator name="${prefix}_actuator">
+                <mechanicalReduction>1</mechanicalReduction>
+            </actuator>
+        </transmission>
+    </xacro:macro>
+<!-- =============================================================================== -->
+<!--  ROS material (change in future)                                                -->
+<!-- =============================================================================== -->
+    <material name="Grey">
+        <color rgba="${107/255} ${107/255} ${107/255} 1.0"/>
+    </material>
+<!-- =============================================================================== -->
+<!--  Link definition                                                                -->
+<!-- =============================================================================== -->
+    <link name="base">
+        <visual>
+            <origin rpy="0 0 0" xyz="0 0 0"/>
+            <geometry>
+                <mesh filename="package://anymal_c_simple_description/meshes/base.dae" scale="1.0 1.0 1.0"/>
+            </geometry>
+        </visual>
+        <collision>
+            <origin rpy="0 0 0" xyz="0 0 0"/>
+            <geometry>
+                <box size="0.58 0.14 0.18"/>
+            </geometry>
+        </collision>
+        <collision>
+            <origin rpy="0 1.57079632679 0" xyz="0.2175 0.07 0"/>
+            <geometry>
+                <cylinder length="0.145" radius="0.09"/>
+            </geometry>
+        </collision>
+        <collision>
+            <origin rpy="0 1.57079632679 0" xyz="-0.2175 0.07 0"/>
+            <geometry>
+                <cylinder length="0.145" radius="0.09"/>
+            </geometry>
+        </collision>
+        <collision>
+            <origin rpy="0 1.57079632679 0" xyz="0.2175 -0.07 0"/>
+            <geometry>
+                <cylinder length="0.145" radius="0.09"/>
+            </geometry>
+        </collision>
+        <collision>
+            <origin rpy="0 1.57079632679 0" xyz="-0.2175 -0.07 0"/>
+            <geometry>
+                <cylinder length="0.145" radius="0.09"/>
+            </geometry>
+        </collision>
+        <!-- Shell self filtering -->
+        <self_filter>
+            <origin rpy="0 0 0" xyz="0 0 0"/>
+            <geometry>
+                <box size="1.05 0.5 0.5"/>
+            </geometry>
+        </self_filter>
+    </link>
+    <!-- Fixed joint to add dummy inertia link -->
+    <joint name="base_to_base_inertia" type="fixed">
+        <parent link="base"/>
+        <child link="base_inertia"/>
+        <origin rpy="0 0 0" xyz="0 0 0"/>
+    </joint>
+    <!-- Dummy inertia link, because KDL cannot have inertia on the base link -->
+    <link name="base_inertia">
+        <inertial>
+            <origin rpy="0 0 0" xyz="-0.018 -0.002 0.024"/>
+            <mass value="6.222"/>
+            <inertia ixx="0.017938806" ixy="0.00387963" ixz="0.001500772" iyy="0.370887745" iyz="6.8963e-05" izz="0.372497653"/>
+        </inertial>
+    </link>
+    <!-- Fixed joint base topshell -->
+    <joint name="base_top_shell" type="fixed">
+        <parent link="base"/>
+        <child link="top_shell"/>
+        <origin rpy="0 0 0" xyz="0 0 0"/>
+    </joint>
+    <!-- Top shell link -->
+    <link name="top_shell">
+        <visual>
+            <origin rpy="0 0 0" xyz="0 0 0"/>
+            <geometry>
+                <mesh filename="package://anymal_c_simple_description/meshes/top_shell.dae" scale="1.0 1.0 1.0"/>
+            </geometry>
+        </visual>
+        <inertial>
+            <origin rpy="0 0 0" xyz="-0.00777 -0.00013 0.06523"/>
+            <mass value="0.534"/>
+            <inertia ixx="0.00664789486" ixy="1.247923e-05" ixz="0.00053990097" iyy="0.02587392411" iyz="3.7614e-07" izz="0.03152303792"/>
+        </inertial>
+    </link>
+    <!-- Fixed joint base topshell -->
+    <joint name="base_bottom_shell" type="fixed">
+        <parent link="base"/>
+        <child link="bottom_shell"/>
+        <origin rpy="0 0 0" xyz="0 0 0"/>
+    </joint>
+    <!-- Bottom shell link -->
+    <link name="bottom_shell">
+        <visual>
+            <origin rpy="0 0 0" xyz="0 0 0"/>
+            <geometry>
+                <mesh filename="package://anymal_c_simple_description/meshes/bottom_shell.dae" scale="1.0 1.0 1.0"/>
+            </geometry>
+        </visual>
+        <inertial>
+            <origin rpy="0 0 0" xyz="-0.00333 1e-05 -0.07705"/>
+            <mass value="1.15"/>
+            <inertia ixx="0.00927353677" ixy="5.41222e-06" ixz="9.039821e-05" iyy="0.06134388239" iyz="2.3042e-07" izz="0.06853531465"/>
+        </inertial>
+    </link>
+    <!-- Fixed joint base remote -->
+    <joint name="base_remote" type="fixed">
+        <parent link="base"/>
+        <child link="remote"/>
+        <origin rpy="0 0 0" xyz="0 0 0"/>
+    </joint>
+    <!-- Remote link -->
+    <link name="remote">
+        <visual>
+            <origin rpy="0 0 0" xyz="0 0 0"/>
+            <geometry>
+                <mesh filename="package://anymal_c_simple_description/meshes/remote.dae" scale="1.0 1.0 1.0"/>
+            </geometry>
+        </visual>
+        <inertial>
+            <origin rpy="0 0 0" xyz="-0.171 0.002 0.096"/>
+            <mass value="0.3262"/>
+            <inertia ixx="0.000528486" ixy="4.547e-05" ixz="1.10327e-05" iyy="0.001165035" iyz="7.4e-07" izz="0.00124026"/>
+        </inertial>
+    </link>
+    <!-- Fixed joint base handle -->
+    <joint name="base_handle" type="fixed">
+        <parent link="base"/>
+        <child link="handle"/>
+        <origin rpy="0 0 0" xyz="0 0 0"/>
+    </joint>
+    <!-- Handle link -->
+    <link name="handle">
+        <visual>
+            <origin rpy="0 0 0" xyz="0 0 0"/>
+            <geometry>
+                <mesh filename="package://anymal_c_simple_description/meshes/handle.dae" scale="1.0 1.0 1.0"/>
+            </geometry>
+        </visual>
+        <inertial>
+            <origin rpy="0 0 0" xyz="0.37801 0.0 0.1372"/>
+            <mass value="0.314"/>
+            <inertia ixx="0.001525739" ixy="0.0" ixz="6.272e-05" iyy="0.00071584" iyz="1e-09" izz="0.001164779"/>
+        </inertial>
+    </link>
+    <!-- Fixed joint base face -->
+    <joint name="base_face_front" type="fixed">
+        <parent link="base"/>
+        <child link="face_front"/>
+        <origin rpy="0 0 -0.0" xyz="0.4145 0 0"/>
+    </joint>
+    <!-- Shell link -->
+    <link name="face_front">
+        <visual>
+            <origin rpy="0 0 0" xyz="0 0 0"/>
+            <geometry>
+                <mesh filename="package://anymal_c_simple_description/meshes/face.dae" scale="1.0 1.0 1.0"/>
+            </geometry>
+        </visual>
+        <collision>
+            <origin rpy="0 0 0" xyz="0.055 0 0"/>
+            <geometry>
+                <box size="0.11 0.14 0.18"/>
+            </geometry>
+        </collision>
+        <collision>
+            <origin rpy="0 1.57079632679 0" xyz="0.055 0.07 0"/>
+            <geometry>
+                <cylinder length="0.11" radius="0.09"/>
+            </geometry>
+        </collision>
+        <collision>
+            <origin rpy="0 1.57079632679 0" xyz="0.055 -0.07 0"/>
+            <geometry>
+                <cylinder length="0.11" radius="0.09"/>
+            </geometry>
+        </collision>
+        <inertial>
+            <origin rpy="0 0 0" xyz="0.042 -0.001 0.004"/>
+            <mass value="0.73"/>
+            <inertia ixx="0.005238611" ixy="1.7609e-05" ixz="7.2167e-05" iyy="0.002643098" iyz="1.9548e-05" izz="0.004325938"/>
+        </inertial>
+    </link>
+    <!-- Camera joint -->
+    <!-- Is located between the two back screw holes at ground level. -->
+    <joint name="face_front_to_depth_camera_front_camera" type="fixed">
+        <parent link="face_front"/>
+        <child link="depth_camera_front_camera"/>
+        <origin rpy="0.0 0.523598775598 0" xyz="0.04715 0.0 -0.0292"/>
+    </joint>
+    <!-- Camera link -->
+    <link name="depth_camera_front_camera">
+        <visual>
+            <origin rpy="0 0 0" xyz="0.0 0.0 0.0"/>
+            <geometry>
+                <mesh filename="package://anymal_c_simple_description/meshes/depth_camera.dae" scale="1.0 1.0 1.0"/>
+            </geometry>
+        </visual>
+        <inertial>
+            <origin rpy="0 0 0" xyz="-0.021 -0.002 0.025"/>
+            <mass value="0.16043"/>
+            <inertia ixx="0.000637051" ixy="0.000484569" ixz="0.000424211" iyy="0.000929402" iyz="5.138e-06" izz="0.000484569"/>
+        </inertial>
+    </link>
+    <!-- Camera parent joint -->
+    <!-- Frame lies on the left ir camera according to any_realsense2_camera urdf. -->
+    <joint name="depth_camera_front_camera_to_camera_parent" type="fixed">
+        <parent link="depth_camera_front_camera"/>
+        <child link="depth_camera_front_camera_parent"/>
+        <origin rpy="0.0 0.0 0.0" xyz="0.0255 0.0175 0.0"/>
+    </joint>
+    <!-- Camera parent link -->
+    <link name="depth_camera_front_camera_parent"/>
+    <!-- Depth optical frame joint -->
+    <joint name="depth_camera_front_camera_parent_to_depth_optical_frame" type="fixed">
+        <parent link="depth_camera_front_camera_parent"/>
+        <child link="depth_camera_front_depth_optical_frame"/>
+        <origin rpy="-1.57079632679 0.0 -1.57079632679" xyz="0.0 0.0 0.0"/>
+    </joint>
+    <!-- Depth optical frame link -->
+    <link name="depth_camera_front_depth_optical_frame"/>
+    <!-- Camera color frame joint -->
+    <joint name="depth_camera_front_camera_parent_to_color_frame" type="fixed">
+        <parent link="depth_camera_front_camera_parent"/>
+        <child link="depth_camera_front_color_frame"/>
+        <origin rpy="0 0 0" xyz="0 0.015 0"/>
+    </joint>
+    <!-- Camera color frame link -->
+    <link name="depth_camera_front_color_frame"/>
+    <!-- Camera color optical joint -->
+    <joint name="depth_camera_front_color_frame_to_color_optical_frame" type="fixed">
+        <parent link="depth_camera_front_color_frame"/>
+        <child link="depth_camera_front_color_optical_frame"/>
+        <origin rpy="-1.57079632679 0.0 -1.57079632679" xyz="0.0 0.0 0.0"/>
+    </joint>
+    <!-- Camera color optical link -->
+    <link name="depth_camera_front_color_optical_frame"/>
+    <!-- Camera joint -->
+    <!-- Is located in the center of the mounting points. -->
+    <joint name="face_front_to_wide_angle_camera_front_camera" type="fixed">
+        <parent link="face_front"/>
+        <child link="wide_angle_camera_front_camera"/>
+        <origin rpy="0 0 0" xyz="0.09850 0.0 0.01497"/>
+    </joint>
+    <!-- Camera link -->
+    <link name="wide_angle_camera_front_camera">
+        <visual>
+            <origin rpy="0 0 0" xyz="0.0 0.0 0.0"/>
+            <geometry>
+                <mesh filename="package://anymal_c_simple_description/meshes/wide_angle_camera.dae" scale="1.0 1.0 1.0"/>
+            </geometry>
+        </visual>
+        <inertial>
+            <origin rpy="0 0 0" xyz="-0.053 -0.001 0.025"/>
+            <mass value="0.287"/>
+            <inertia ixx="0.000559232" ixy="1.6875e-05" ixz="0.000423761" iyy="0.000946504" iyz="1.3234e-07" izz="0.000493052"/>
+        </inertial>
+    </link>
+    <!-- Camera parent joint -->
+    <joint name="wide_angle_camera_front_camera_to_camera_parent" type="fixed">
+        <parent link="wide_angle_camera_front_camera"/>
+        <child link="wide_angle_camera_front_camera_parent"/>
+        <origin rpy="-1.57079632679 0.0 -1.57079632679" xyz="0.0 0.0 0.0"/>
+    </joint>
+    <!-- Camera parent link -->
+    <link name="wide_angle_camera_front_camera_parent"/>
+    <!-- Fixed joint base face -->
+    <joint name="base_face_rear" type="fixed">
+        <parent link="base"/>
+        <child link="face_rear"/>
+        <origin rpy="0 0 3.14159265359" xyz="-0.4145 0 0"/>
+    </joint>
+    <!-- Shell link -->
+    <link name="face_rear">
+        <visual>
+            <origin rpy="0 0 0" xyz="0 0 0"/>
+            <geometry>
+                <mesh filename="package://anymal_c_simple_description/meshes/face.dae" scale="1.0 1.0 1.0"/>
+            </geometry>
+        </visual>
+        <collision>
+            <origin rpy="0 0 0" xyz="0.055 0 0"/>
+            <geometry>
+                <box size="0.11 0.14 0.18"/>
+            </geometry>
+        </collision>
+        <collision>
+            <origin rpy="0 1.57079632679 0" xyz="0.055 0.07 0"/>
+            <geometry>
+                <cylinder length="0.11" radius="0.09"/>
+            </geometry>
+        </collision>
+        <collision>
+            <origin rpy="0 1.57079632679 0" xyz="0.055 -0.07 0"/>
+            <geometry>
+                <cylinder length="0.11" radius="0.09"/>
+            </geometry>
+        </collision>
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
Commit message: fixing gazebo bringup

File: aww_description/urdf/anymal_with_wheels.urdf.xacro (robot description, xacro)
@@ -54,5 +54,5 @@
             <inertial>
                 <origin xyz="0 0 0" rpy="0 0 0"/>
-                <mass value="0.477"/>
+                <mass value="0.2"/>
                 <inertia
                     ixx="0.0013" ixy="0" ixz="0"
@@ -310,5 +310,5 @@
         <inertial>
             <origin rpy="0 0 0" xyz="0.042 -0.001 0.004"/>
-            <mass value="0.73"/>
+            <mass value="12.73"/>
             <inertia ixx="0.005238611" ixy="1.7609e-05" ixz="7.2167e-05" iyy="0.002643098" iyz="1.9548e-05" izz="0.004325938"/>
         </inertial>
@@ -615,5 +615,5 @@
         <inertial>
             <origin rpy="0 0 0" xyz="0.00948 -0.00948 0.1468"/>
-            <mass value="0.25"/>
+            <mass value="0.15"/>
             <inertia ixx="0.00317174097" ixy="2.63048e-06" ixz="6.815581e-05" iyy="0.00317174092" iyz="6.815583e-05" izz="8.319196e-05"/>
         </inertial>
@@ -860,5 +860,5 @@
         <inertial>
             <origin rpy="0 0 0" xyz="0.00948 0.00948 0.1468"/>
-            <mass value="0.25"/>
+            <mass value="0.15"/>
             <inertia ixx="0.00317174097" ixy="-2.63048e-06" ixz="6.815581e-05" iyy="0.00317174092" iyz="-6.815583e-05" izz="8.319196e-05"/>
         </inertial>
@@ -1105,5 +1105,5 @@
         <inertial>
             <origin rpy="0 0 0" xyz="-0.00948 -0.00948 0.1468"/>
-            <mass value="0.25"/>
+            <mass value="0.15"/>
             <inertia ixx="0.00317174097" ixy="-2.63048e-06" ixz="-6.815581e-05" iyy="0.00317174092" iyz="6.815583e-05" izz="8.319196e-05"/>
         </inertial>
@@ -1350,5 +1350,5 @@
         <inertial>
             <origin rpy="0 0 0" xyz="-0.00948 0.00948 0.1468"/>
-            <mass value="0.25"/>
+            <mass value="0.15"/>
             <inertia ixx="0.00317174097" ixy="2.63048e-06" ixz="-6.815581e-05" iyy="0.00317174092" iyz="-6.815583e-05" izz="8.319196e-05"/>
         </inertial>
