Commit message: changes in description, add velodyne, and differential controller

File: aww_description/urdf/anymal_with_wheels.urdf (robot description, URDF)
Before this commit: robot anymal_with_wheels, 82 links, 81 joints
Links:
- removed link handle
- removed link lidar
- added link velodyne, mass 0.01; visual mesh filename=package://velodyne_description/meshes/VLP16_scan.dae
- added link velodyne_base_link, mass 0.83; collision cylinder length=0.0717 radius=0.0516; visual mesh filename=package://velodyne_description/meshes/VLP16_base_1.dae
Joints:
- removed joint base_handle
- removed joint lidar_cage_to_lidar
- added joint velodyne_base_mount_joint: type fixed, parent lidar_cage, child velodyne_base_link, origin xyz=0 0 0.03 rpy=0 0 0
- added joint velodyne_base_scan_joint: type fixed, parent velodyne_base_link, child velodyne, origin xyz=0 0 0.0377 rpy=0 0 0
- joint base_to_lidar_cage: origin xyz=-0.364 0.0 0.0735 rpy=0 0 0 -> xyz=0.364 0.0 0.0635 rpy=0 0 0

File: aww_description/urdf/anymal_with_wheels.urdf.xacro (robot description, xacro)
@@ -217,12 +217,13 @@
         </inertial>
     </link>
+    <!-- We use the velodyne in front -->
     <!-- Fixed joint base handle -->
-    <joint name="base_handle" type="fixed">
+    <!-- joint name="base_handle" type="fixed">
         <parent link="base"/>
         <child link="handle"/>
         <origin rpy="0 0 0" xyz="0 0 0"/>
-    </joint>
+    </joint-->
     <!-- Handle link -->
-    <link name="handle">
+    <!--link name="handle">
         <visual>
             <origin rpy="0 0 0" xyz="0 0 0"/>
@@ -236,5 +237,5 @@
             <inertia ixx="0.001525739" ixy="0.0" ixz="6.272e-05" iyy="0.00071584" iyz="1e-09" izz="0.001164779"/>
         </inertial>
-    </link>
+    </link-->
     <!-- Fixed joint base face -->
     <joint name="base_face_front" type="fixed">
@@ -647,50 +648,4 @@
     <!-- Camera color optical link -->
     <link name="depth_camera_right_color_optical_frame"/>
-    <!-- parent to cage joint, located between mounting plate on trunk and the cage -->
-    <joint name="base_to_lidar_cage" type="fixed">
-        <parent link="base"/>
-        <child link="lidar_cage"/>
-        <origin rpy="0 0 0" xyz="-0.364 0.0 0.0735"/>
-    </joint>
-    <!-- Velodyne cage link -->
-    <link name="lidar_cage">
-        <visual>
-            <origin rpy="0.0 0.0 0.0" xyz="0.0 0.0 0.0"/>
-            <geometry>
-                <mesh filename="package://anymal_c_simple_description/meshes/lidar_cage.dae" scale="1.0 1.0 1.0"/>
-            </geometry>
-        </visual>
-        <collision>
-            <origin rpy="0 0 0" xyz="0 0 0.06"/>
-            <geometry>
-                <cylinder length="0.12" radius="0.07"/>
-            </geometry>
-        </collision>
-        <inertial>
-            <origin rpy="0.0 0.0 0.0" xyz="0.002 0.0 0.099"/>
-            <mass value="0.545"/>
-            <inertia ixx="0.003156254" ixy="0.0" ixz="1.0992e-05" iyy="0.002357216" iyz="0.0" izz="0.001326455"/>
-        </inertial>
-    </link>
-    <!-- parent to sensor joint -->
-    <joint name="lidar_cage_to_lidar" type="fixed">
-        <parent link="lidar_cage"/>
-        <child link="lidar"/>
-        <origin rpy="0.0 0.0 -1.57079632679" xyz="0.0 0.0 0.0687"/>
-    </joint>
-    <!-- Velodyne sensor link -->
-    <link name="lidar">
-        <inertial>
-            <origin rpy="0.0 0.0 0.0" xyz="-0.012 0.001 -0.008"/>
-            <mass value="0.695"/>
-            <inertia ixx="0.000846765" ixy="6.9565e-05" ixz="0.00027111" iyy="0.001367583" iyz="5.8984e-05" izz="0.001363673"/>
-        </inertial>
-        <visual>
-            <origin xyz="0 0 0"/>
-            <geometry>
-                <mesh filename="package://anymal_c_simple_description/meshes/lidar.dae"/>
-            </geometry>
-        </visual>
-    </link>
     <!-- joint base HAA -->
     <joint name="base_LF_HAA" type="fixed">
@@ -1727,3 +1682,7 @@
 <!-- =============================================================================== -->
     <xacro:include filename="$(find aww_description)/urdf/aww.gazebo" />
+<!-- =============================================================================== -->
+<!--  Import acessories                                                              -->
+<!-- =============================================================================== -->
+    <xacro:include filename="$(find aww_description)/urdf/acessories.urdf.xacro" />
 </robot>

Commit message: refactoring the robot urdf and remove camera links and joints

File: aww_description/urdf/anymal_with_wheels.urdf (robot description, URDF)
Before this commit: robot aww, 82 links, 81 joints
Links:
- removed link depth_camera_front_camera
- removed link depth_camera_front_camera_parent
- removed link depth_camera_front_color_frame
- removed link depth_camera_front_color_optical_frame
- removed link depth_camera_front_depth_optical_frame
- removed link depth_camera_left_camera
- removed link depth_camera_left_camera_parent
- removed link depth_camera_left_color_frame
- removed link depth_camera_left_color_optical_frame
- removed link depth_camera_left_depth_optical_frame
- removed link depth_camera_rear_camera
- removed link depth_camera_rear_camera_parent
- removed link depth_camera_rear_color_frame
- removed link depth_camera_rear_color_optical_frame
- removed link depth_camera_rear_depth_optical_frame
- removed link depth_camera_right_camera
- removed link depth_camera_right_camera_parent
- removed link depth_camera_right_color_frame
- removed link depth_camera_right_color_optical_frame
- removed link depth_camera_right_depth_optical_frame
- removed link wide_angle_camera_front_camera
- removed link wide_angle_camera_front_camera_parent
- removed link wide_angle_camera_rear_camera
- removed link wide_angle_camera_rear_camera_parent
Joints:
- removed joint base_to_depth_camera_left_camera
- removed joint base_to_depth_camera_right_camera
- removed joint depth_camera_front_camera_parent_to_color_frame
- removed joint depth_camera_front_camera_parent_to_depth_optical_frame
- removed joint depth_camera_front_camera_to_camera_parent
- removed joint depth_camera_front_color_frame_to_color_optical_frame
- removed joint depth_camera_left_camera_parent_to_color_frame
- removed joint depth_camera_left_camera_parent_to_depth_optical_frame
- removed joint depth_camera_left_camera_to_camera_parent
- removed joint depth_camera_left_color_frame_to_color_optical_frame
- removed joint depth_camera_rear_camera_parent_to_color_frame
- removed joint depth_camera_rear_camera_parent_to_depth_optical_frame
- removed joint depth_camera_rear_camera_to_camera_parent
- removed joint depth_camera_rear_color_frame_to_color_optical_frame
- removed joint depth_camera_right_camera_parent_to_color_frame
- removed joint depth_camera_right_camera_parent_to_depth_optical_frame
- removed joint depth_camera_right_camera_to_camera_parent
- removed joint depth_camera_right_color_frame_to_color_optical_frame
- removed joint face_front_to_depth_camera_front_camera
- removed joint face_front_to_wide_angle_camera_front_camera
- removed joint face_rear_to_depth_camera_rear_camera
- removed joint face_rear_to_wide_angle_camera_rear_camera
- removed joint wide_angle_camera_front_camera_to_camera_parent
- removed joint wide_angle_camera_rear_camera_to_camera_parent

File: aww_description/urdf/anymal_with_wheels.urdf.xacro (robot description, xacro)
@@ -276,87 +276,4 @@
         </inertial>
     </link>
-    <!-- Camera joint -->
-    <!-- Is located between the two back screw holes at ground level. -->
-    <joint name="face_front_to_depth_camera_front_camera" type="fixed">
-        <parent link="face_front"/>
-        <child link="depth_camera_front_camera"/>
-        <origin rpy="0.0 0.523598775598 0" xyz="0.04715 0.0 -0.0292"/>
-    </joint>
-    <!-- Camera link -->
-    <link name="depth_camera_front_camera">
-        <visual>
-            <origin rpy="0 0 0" xyz="0.0 0.0 0.0"/>
-            <geometry>
-                <mesh filename="package://anymal_c_simple_description/meshes/depth_camera.dae" scale="1.0 1.0 1.0"/>
-            </geometry>
-        </visual>
-        <inertial>
-            <origin rpy="0 0 0" xyz="-0.021 -0.002 0.025"/>
-            <mass value="0.16043"/>
-            <inertia ixx="0.000637051" ixy="0.000484569" ixz="0.000424211" iyy="0.000929402" iyz="5.138e-06" izz="0.000484569"/>
-        </inertial>
-    </link>
-    <!-- Camera parent joint -->
-    <!-- Frame lies on the left ir camera according to any_realsense2_camera urdf. -->
-    <joint name="depth_camera_front_camera_to_camera_parent" type="fixed">
-        <parent link="depth_camera_front_camera"/>
-        <child link="depth_camera_front_camera_parent"/>
-        <origin rpy="0.0 0.0 0.0" xyz="0.0255 0.0175 0.0"/>
-    </joint>
-    <!-- Camera parent link -->
-    <link name="depth_camera_front_camera_parent"/>
-    <!-- Depth optical frame joint -->
-    <joint name="depth_camera_front_camera_parent_to_depth_optical_frame" type="fixed">
-        <parent link="depth_camera_front_camera_parent"/>
-        <child link="depth_camera_front_depth_optical_frame"/>
-        <origin rpy="-1.57079632679 0.0 -1.57079632679" xyz="0.0 0.0 0.0"/>
-    </joint>
-    <!-- Depth optical frame link -->
-    <link name="depth_camera_front_depth_optical_frame"/>
-    <!-- Camera color frame joint -->
-    <joint name="depth_camera_front_camera_parent_to_color_frame" type="fixed">
-        <parent link="depth_camera_front_camera_parent"/>
-        <child link="depth_camera_front_color_frame"/>
-        <origin rpy="0 0 0" xyz="0 0.015 0"/>
-    </joint>
-    <!-- Camera color frame link -->
-    <link name="depth_camera_front_color_frame"/>
-    <!-- Camera color optical joint -->
-    <joint name="depth_camera_front_color_frame_to_color_optical_frame" type="fixed">
-        <parent link="depth_camera_front_color_frame"/>
-        <child link="depth_camera_front_color_optical_frame"/>
-        <origin rpy="-1.57079632679 0.0 -1.57079632679" xyz="0.0 0.0 0.0"/>
-    </joint>
-    <!-- Camera color optical link -->
-    <link name="depth_camera_front_color_optical_frame"/>
-    <!-- Camera joint -->
-    <!-- Is located in the center of the mounting points. -->
-    <joint name="face_front_to_wide_angle_camera_front_camera" type="fixed">
-        <parent link="face_front"/>
-        <child link="wide_angle_camera_front_camera"/>
-        <origin rpy="0 0 0" xyz="0.09850 0.0 0.01497"/>
-    </joint>
-    <!-- Camera link -->
-    <link name="wide_angle_camera_front_camera">
-        <visual>
-            <origin rpy="0 0 0" xyz="0.0 0.0 0.0"/>
-            <geometry>
-                <mesh filename="package://anymal_c_simple_description/meshes/wide_angle_camera.dae" scale="1.0 1.0 1.0"/>
-            </geometry>
-        </visual>
-        <inertial>
-            <origin rpy="0 0 0" xyz="-0.053 -0.001 0.025"/>
-            <mass value="0.287"/>
-            <inertia ixx="0.000559232" ixy="1.6875e-05" ixz="0.000423761" iyy="0.000946504" iyz="1.3234e-07" izz="0.000493052"/>
-        </inertial>
-    </link>
-    <!-- Camera parent joint -->
-    <joint name="wide_angle_camera_front_camera_to_camera_parent" type="fixed">
-        <parent link="wide_angle_camera_front_camera"/>
-        <child link="wide_angle_camera_front_camera_parent"/>
-        <origin rpy="-1.57079632679 0.0 -1.57079632679" xyz="0.0 0.0 0.0"/>
-    </joint>
-    <!-- Camera parent link -->
-    <link name="wide_angle_camera_front_camera_parent"/>
     <!-- Fixed joint base face -->
     <joint name="base_face_rear" type="fixed">
@@ -397,87 +314,4 @@
         </inertial>
     </link>
-    <!-- Camera joint -->
-    <!-- Is located between the two back screw holes at ground level. -->
-    <joint name="face_rear_to_depth_camera_rear_camera" type="fixed">
-        <parent link="face_rear"/>
-        <child link="depth_camera_rear_camera"/>
-        <origin rpy="0.0 0.523598775598 0" xyz="0.04715 0.0 -0.0292"/>
-    </joint>
-    <!-- Camera link -->
-    <link name="depth_camera_rear_camera">
-        <visual>
-            <origin rpy="0 0 0" xyz="0.0 0.0 0.0"/>
-            <geometry>
-                <mesh filename="package://anymal_c_simple_description/meshes/depth_camera.dae" scale="1.0 1.0 1.0"/>
-            </geometry>
-        </visual>
-        <inertial>
-            <origin rpy="0 0 0" xyz="-0.021 -0.002 0.025"/>
-            <mass value="0.16043"/>
-            <inertia ixx="0.000637051" ixy="0.000484569" ixz="0.000424211" iyy="0.000929402" iyz="5.138e-06" izz="0.000484569"/>
-        </inertial>
-    </link>
-    <!-- Camera parent joint -->
-    <!-- Frame lies on the left ir camera according to any_realsense2_camera urdf. -->
-    <joint name="depth_camera_rear_camera_to_camera_parent" type="fixed">
-        <parent link="depth_camera_rear_camera"/>
-        <child link="depth_camera_rear_camera_parent"/>
-        <origin rpy="0.0 0.0 0.0" xyz="0.0255 0.0175 0.0"/>
-    </joint>
-    <!-- Camera parent link -->
-    <link name="depth_camera_rear_camera_parent"/>
-    <!-- Depth optical frame joint -->
-    <joint name="depth_camera_rear_camera_parent_to_depth_optical_frame" type="fixed">
-        <parent link="depth_camera_rear_camera_parent"/>
-        <child link="depth_camera_rear_depth_optical_frame"/>
-        <origin rpy="-1.57079632679 0.0 -1.57079632679" xyz="0.0 0.0 0.0"/>
-    </joint>
-    <!-- Depth optical frame link -->
-    <link name="depth_camera_rear_depth_optical_frame"/>
-    <!-- Camera color frame joint -->
-    <joint name="depth_camera_rear_camera_parent_to_color_frame" type="fixed">
-        <parent link="depth_camera_rear_camera_parent"/>
-        <child link="depth_camera_rear_color_frame"/>
-        <origin rpy="0 0 0" xyz="0 0.015 0"/>
-    </joint>
-    <!-- Camera color frame link -->
-    <link name="depth_camera_rear_color_frame"/>
-    <!-- Camera color optical joint -->
-    <joint name="depth_camera_rear_color_frame_to_color_optical_frame" type="fixed">
-        <parent link="depth_camera_rear_color_frame"/>
-        <child link="depth_camera_rear_color_optical_frame"/>
-        <origin rpy="-1.57079632679 0.0 -1.57079632679" xyz="0.0 0.0 0.0"/>
-    </joint>
-    <!-- Camera color optical link -->
-    <link name="depth_camera_rear_color_optical_frame"/>
-    <!-- Camera joint -->
-    <!-- Is located in the center of the mounting points. -->
-    <joint name="face_rear_to_wide_angle_camera_rear_camera" type="fixed">
-        <parent link="face_rear"/>
-        <child link="wide_angle_camera_rear_camera"/>
-        <origin rpy="0 0 0" xyz="0.09850 0.0 0.01497"/>
-    </joint>
-    <!-- Camera link -->
-    <link name="wide_angle_camera_rear_camera">
-        <visual>
-            <origin rpy="0 0 0" xyz="0.0 0.0 0.0"/>
-            <geometry>
-                <mesh filename="package://anymal_c_simple_description/meshes/wide_angle_camera.dae" scale="1.0 1.0 1.0"/>
-            </geometry>
-        </visual>
-        <inertial>
-            <origin rpy="0 0 0" xyz="-0.053 -0.001 0.025"/>
-            <mass value="0.287"/>
-            <inertia ixx="0.000559232" ixy="1.6875e-05" ixz="0.000423761" iyy="0.000946504" iyz="1.3234e-07" izz="0.000493052"/>
-        </inertial>
-    </link>
-    <!-- Camera parent joint -->
-    <joint name="wide_angle_camera_rear_camera_to_camera_parent" type="fixed">
-        <parent link="wide_angle_camera_rear_camera"/>
-        <child link="wide_angle_camera_rear_camera_parent"/>
-        <origin rpy="-1.57079632679 0.0 -1.57079632679" xyz="0.0 0.0 0.0"/>
-    </joint>
-    <!-- Camera parent link -->
-    <link name="wide_angle_camera_rear_camera_parent"/>
     <!-- Fixed joint base battery -->
     <joint name="base_battery" type="fixed">
@@ -540,112 +374,4 @@
         <origin rpy="0.0 0.0 1.57079632679" xyz="0.2488 0.00835 0.04628"/>
     </joint>
-    <!-- Camera joint -->
-    <!-- Is located between the two back screw holes at ground level. -->
-    <joint name="base_to_depth_camera_left_camera" type="fixed">
-        <parent link="base"/>
-        <child link="depth_camera_left_camera"/>
-        <origin rpy="0.0 0.523598775598 1.57079632679" xyz="0.0 0.07646 0.02905"/>
-    </joint>
-    <!-- Camera link -->
-    <link name="depth_camera_left_camera">
-        <visual>
-            <origin rpy="0 0 0" xyz="0.0 0.0 0.0"/>
-            <geometry>
-                <mesh filename="package://anymal_c_simple_description/meshes/depth_camera.dae" scale="1.0 1.0 1.0"/>
-            </geometry>
-        </visual>
-        <inertial>
-            <origin rpy="0 0 0" xyz="-0.021 -0.002 0.025"/>
-            <mass value="0.16043"/>
-            <inertia ixx="0.000637051" ixy="0.000484569" ixz="0.000424211" iyy="0.000929402" iyz="5.138e-06" izz="0.000484569"/>
-        </inertial>
-    </link>
-    <!-- Camera parent joint -->
-    <!-- Frame lies on the left ir camera according to any_realsense2_camera urdf. -->
-    <joint name="depth_camera_left_camera_to_camera_parent" type="fixed">
-        <parent link="depth_camera_left_camera"/>
-        <child link="depth_camera_left_camera_parent"/>
-        <origin rpy="0.0 0.0 0.0" xyz="0.0255 0.0175 0.0"/>
-    </joint>
-    <!-- Camera parent link -->
-    <link name="depth_camera_left_camera_parent"/>
-    <!-- Depth optical frame joint -->
-    <joint name="depth_camera_left_camera_parent_to_depth_optical_frame" type="fixed">
-        <parent link="depth_camera_left_camera_parent"/>
-        <child link="depth_camera_left_depth_optical_frame"/>
-        <origin rpy="-1.57079632679 0.0 -1.57079632679" xyz="0.0 0.0 0.0"/>
-    </joint>
-    <!-- Depth optical frame link -->
-    <link name="depth_camera_left_depth_optical_frame"/>
-    <!-- Camera color frame joint -->
-    <joint name="depth_camera_left_camera_parent_to_color_frame" type="fixed">
-        <parent link="depth_camera_left_camera_parent"/>
-        <child link="depth_camera_left_color_frame"/>
-        <origin rpy="0 0 0" xyz="0 0.015 0"/>
-    </joint>
-    <!-- Camera color frame link -->
-    <link name="depth_camera_left_color_frame"/>
-    <!-- Camera color optical joint -->
-    <joint name="depth_camera_left_color_frame_to_color_optical_frame" type="fixed">
-        <parent link="depth_camera_left_color_frame"/>
-        <child link="depth_camera_left_color_optical_frame"/>
-        <origin rpy="-1.57079632679 0.0 -1.57079632679" xyz="0.0 0.0 0.0"/>
-    </joint>
-    <!-- Camera color optical link -->
-    <link name="depth_camera_left_color_optical_frame"/>
-    <!-- Camera joint -->
-    <!-- Is located between the two back screw holes at ground level. -->
-    <joint name="base_to_depth_camera_right_camera" type="fixed">
-        <parent link="base"/>
-        <child link="depth_camera_right_camera"/>
-        <origin rpy="0.0 0.523598775598 -1.57079632679" xyz="0.0 -0.07646 0.02905"/>
-    </joint>
-    <!-- Camera link -->
-    <link name="depth_camera_right_camera">
-        <visual>
-            <origin rpy="0 0 0" xyz="0.0 0.0 0.0"/>
-            <geometry>
-                <mesh filename="package://anymal_c_simple_description/meshes/depth_camera.dae" scale="1.0 1.0 1.0"/>
-            </geometry>
-        </visual>
-        <inertial>
-            <origin rpy="0 0 0" xyz="-0.021 -0.002 0.025"/>
-            <mass value="0.16043"/>
-            <inertia ixx="0.000637051" ixy="0.000484569" ixz="0.000424211" iyy="0.000929402" iyz="5.138e-06" izz="0.000484569"/>
-        </inertial>
-    </link>
-    <!-- Camera parent joint -->
-    <!-- Frame lies on the left ir camera according to any_realsense2_camera urdf. -->
-    <joint name="depth_camera_right_camera_to_camera_parent" type="fixed">
-        <parent link="depth_camera_right_camera"/>
-        <child link="depth_camera_right_camera_parent"/>
-        <origin rpy="0.0 0.0 0.0" xyz="0.0255 0.0175 0.0"/>
-    </joint>
-    <!-- Camera parent link -->
-    <link name="depth_camera_right_camera_parent"/>
-    <!-- Depth optical frame joint -->
-    <joint name="depth_camera_right_camera_parent_to_depth_optical_frame" type="fixed">
-        <parent link="depth_camera_right_camera_parent"/>
-        <child link="depth_camera_right_depth_optical_frame"/>
-        <origin rpy="-1.57079632679 0.0 -1.57079632679" xyz="0.0 0.0 0.0"/>
-    </joint>
-    <!-- Depth optical frame link -->
-    <link name="depth_camera_right_depth_optical_frame"/>
-    <!-- Camera color frame joint -->
-    <joint name="depth_camera_right_camera_parent_to_color_frame" type="fixed">
-        <parent link="depth_camera_right_camera_parent"/>
-        <child link="depth_camera_right_color_frame"/>
-        <origin rpy="0 0 0" xyz="0 0.015 0"/>
-    </joint>
-    <!-- Camera color frame link -->
-    <link name="depth_camera_right_color_frame"/>
-    <!-- Camera color optical joint -->
-    <joint name="depth_camera_right_color_frame_to_color_optical_frame" type="fixed">
-        <parent link="depth_camera_right_color_frame"/>
-        <child link="depth_camera_right_color_optical_frame"/>
-        <origin rpy="-1.57079632679 0.0 -1.57079632679" xyz="0.0 0.0 0.0"/>
-    </joint>
-    <!-- Camera color optical link -->
-    <link name="depth_camera_right_color_optical_frame"/>
     <!-- joint base HAA -->
     <joint name="base_LF_HAA" type="fixed">

Commit message: changes to incorporate the navigation

File: aww_description/urdf/anymal_with_wheels.urdf (robot description, URDF)
Before this commit: robot aww, 58 links, 57 joints
Links:
- link LF_LEG: mass 0.25 -> 0.15
- link LF_wheel_link: mass 0.477 -> 0.2
- link LH_LEG: mass 0.25 -> 0.15
- link LH_wheel_link: mass 0.477 -> 0.2
- link RF_LEG: mass 0.25 -> 0.15
- link RF_wheel_link: mass 0.477 -> 0.2
- link RH_LEG: mass 0.25 -> 0.15
- link RH_wheel_link: mass 0.477 -> 0.2
- link face_rear: mass 0.73 -> 12.73
